Commit message: User Control Setup

File: src/game_gz/urdf_police/gazebo.xacro (robot description, xacro)
@@ -11,6 +11,27 @@
             <wheel_separation>0.5</wheel_separation>
             <wheel_radius>0.05</wheel_radius>
-            <topic>cmd_vel</topic>
+            <topic>/police/cmd_vel</topic>
         </plugin>
     </gazebo>
+    <gazebo reference="pols_camera">
+        <sensor name="camera" type="camera">
+            <pose>0 0 0 0 0 0</pose>
+            <always_on>true</always_on>
+            <update_rate>30.0</update_rate>
+            <visualize>true</visualize>
+            <topic>/police/camera/image</topic>
+            <camera>
+                <horizontal_fov>1.089</horizontal_fov>
+                <image>
+                    <width>640</width>
+                    <height>480</height>
+                    <format>R8G8B8</format>
+                </image>
+                <clip>
+                    <near>0.05</near>
+                    <far>8.0</far>
+                </clip>
+            </camera>
+        </sensor>
+    </gazebo>
 </robot>

File: src/game_gz/urdf_police/properties.xacro (robot description, xacro)
@@ -13,10 +13,10 @@
     <xacro:property name="wheel_length" value="0.1"/>
     <xacro:property name="head_radius" value="0.2"/>
-    <xacro:property name="base_mass" value="3.0"/>
-    <xacro:property name="leg_mass" value="3.0"/>
+    <xacro:property name="base_mass" value="1.0"/>
+    <xacro:property name="leg_mass" value="1.0"/>
     <xacro:property name="pad_mass" value="5.0"/>
     <xacro:property name="wheel_mass" value="3.0"/>
     <xacro:property name="iwheel_mass" value="2.0"/>
-    <xacro:property name="head_mass" value="1.0"/>
+    <xacro:property name="head_mass" value="0.5"/>
     <xacro:property name="eye_socket_mass" value="0.1"/>
     <xacro:property name="eyeball_mass" value="0.05"/>

File: src/game_gz/urdf_police/robot_vtwo.urdf (robot description, URDF)
Before this commit: robot chitti_vtwo, 17 links, 16 joints
Links:
- added link pols_camera, mass 0.05; collision sphere radius=0.05; visual sphere radius=0.05
- link base_link: mass 5.0 -> 1.0
- link head: mass 1.0 -> 0.5
- link iwheel1: mass 0.05 -> 2.0
- link iwheel2: mass 0.05 -> 2.0
- link iwheel3: mass 0.05 -> 2.0
- link iwheel4: mass 0.05 -> 2.0
- link leg_l: mass 0.5 -> 1.0
- link leg_r: mass 0.5 -> 1.0
- link pad_l: mass 0.3 -> 5.0
- link pad_r: mass 0.3 -> 5.0
- link wheel1: mass 0.2 -> 3.0
- link wheel2: mass 0.2 -> 3.0
- link wheel3: mass 0.2 -> 3.0
- link wheel4: mass 0.2 -> 3.0
Joints:
- added joint ceye_joint: type fixed, parent base_link, child pols_camera, origin xyz=0.2 0 0 rpy=0 0 0
- joint leg_joint_l: axis 0 1 0 -> (none); limit lower=-0.5 upper=0.5 effort=100.0 velocity=3.14 -> (none); type revolute -> fixed
- joint leg_joint_r: axis 0 1 0 -> (none); limit lower=-0.5 upper=0.5 effort=100.0 velocity=3.14 -> (none); type revolute -> fixed
- joint wheel1_joint: axis 0 0 1 -> 0 0 -1
- joint wheel2_joint: axis 0 0 1 -> 0 0 -1
- joint wheel3_joint: axis 0 0 1 -> 0 0 -1
- joint wheel4_joint: axis 0 0 1 -> 0 0 -1

File: src/game_gz/urdf_police/robot_vtwo.xacro (robot description, xacro)
@@ -19,4 +19,23 @@
         </collision>
     </link>
+    <link name="pols_camera">
+        <xacro:default_inertial mass="${eyeball_mass}"/>
+        <visual>
+            <geometry>
+                <sphere radius="${head_radius/4}" />
+            </geometry>
+            <material name="white" />
+        </visual>
+        <collision>
+            <geometry>
+                <sphere radius="${head_radius/4}" />
+            </geometry>
+        </collision>
+    </link>
+    <joint name="ceye_joint" type="fixed">
+        <parent link="base_link"/>
+        <child link="pols_camera"/>
+        <origin rpy="0 0 0" xyz="0.2 0 0"/>
+    </joint>
     <xacro:leg_assembly prefix="l" y_offset="-0.25"/>
     <xacro:leg_assembly prefix="r" y_offset="0.25"/>

File: src/game_gz/urdf_thief/gazebo.xacro (robot description, xacro)
@@ -9,6 +9,27 @@
             <wheel_separation>0.7</wheel_separation>
             <wheel_radius>0.04</wheel_radius>
-            <topic>cmd_vel</topic>
+            <topic>/thief/cmd_vel</topic>
         </plugin>
     </gazebo>
+    <gazebo reference="thief_camera">
+        <sensor name="camera" type="camera">
+            <pose>0 0 0 0 0 0</pose>
+            <always_on>true</always_on>
+            <update_rate>30.0</update_rate>
+            <visualize>true</visualize>
+            <topic>/thief/camera/image</topic>
+            <camera>
+                <horizontal_fov>1.089</horizontal_fov>
+                <image>
+                    <width>640</width>
+                    <height>480</height>
+                    <format>R8G8B8</format>
+                </image>
+                <clip>
+                    <near>0.05</near>
+                    <far>8.0</far>
+                </clip>
+            </camera>
+        </sensor>
+    </gazebo>
 </robot>

File: src/game_gz/urdf_thief/tuktuk.urdf (robot description, URDF)
Before this commit: robot tuktuk, 22 links, 21 joints
Links:
- added link stand, mass 0.001; collision cylinder length=0.5 radius=0.01; visual cylinder length=0.5 radius=0.01
- added link thief_camera, mass 0.001; collision sphere radius=0.06; visual sphere radius=0.05
Joints:
- added joint cam_joint: type fixed, parent stand, child thief_camera, origin xyz=0 0 0.25 rpy=0 0 0
- added joint stand_joint: type fixed, parent chassis, child stand, origin xyz=0 0 0.28 rpy=0 0 0

File: src/game_gz/urdf_thief/tuktuk.xacro (robot description, xacro)
@@ -22,14 +22,42 @@
         </collision>
     </link>
+    <link name="stand">
+        <xacro:zero_inertial/>
+        <visual>
+            <geometry>
+                <cylinder radius="0.01" length='0.5'/>
+            </geometry>
+            <material name="white" />
+        </visual>
+        <collision>
+            <geometry>
+                <cylinder radius="0.01" length='0.5'/>
+            </geometry>
+        </collision>
+    </link>
+    <joint name="stand_joint" type="fixed">
+        <parent link="chassis"/>
+        <child link="stand"/>
+        <origin rpy="0 0 0" xyz="0 0 0.28"/>
+    </joint>
+    <link name="thief_camera">
+        <xacro:zero_inertial/>
+        <visual>
+            <geometry>
+                <sphere radius="0.05" />
+            </geometry>
+            <material name="blue" />
+        </visual>
+        <collision>
+            <geometry>
+                <sphere radius="0.06" />
+            </geometry>
+        </collision>
+    </link>
+    <joint name="cam_joint" type="fixed">
+        <parent link="stand"/>
+        <child link="thief_camera"/>
+        <origin rpy="0 0 0" xyz="0 0 0.25"/>
+    </joint>
     <xacro:main_assembly/>
 </robot>
-<!-- I used xacro to make this bot coz its easy to modify this way.
-    Most of the dimensions and origin of links are in properties.xacro.
-    macros.xacro has all the macros used in main_assembly macro itself.
-    materials.xacro has the colors(materials).
-    gazebo.xacro has the diff drive plugin used in task 4b.
-    I used chassis instead of base_link.
-    The original tuktuk is in MiniTask.
-    More logic is inside macros.xacro
-    KDL might throw a warning coz kdl does not support root link with inertia,
-    but i did not create a dummy link coz without inertial and collision, chassis will be invisible in gazebo-->

Commit message: v1.0 done

File: src/game_gz/urdf_police/gazebo.xacro (robot description, xacro)
@@ -35,3 +35,12 @@
         </sensor>
     </gazebo>
+    <gazebo reference="catch">
+        <sensor name="contact_sensor" type="contact">
+            <always_on>true</always_on>
+            <update_rate>30</update_rate>
+            <contact>
+                <collision>base_link_fixed_joint_lump__busted_collision_1</collision>
+            </contact>
+        </sensor>
+    </gazebo>
 </robot>

File: src/game_gz/urdf_police/materials.xacro (robot description, xacro)
@@ -16,3 +16,6 @@
                 <color rgba="1 1 0 1"/>
     </material>
+    <material name="red">
+                <color rgba="1 0 0 1"/>
+    </material>
 </robot>

File: src/game_gz/urdf_police/robot_vtwo.xacro (robot description, xacro)
@@ -19,4 +19,23 @@
         </collision>
     </link>
+    <link name="catch">
+        <xacro:default_inertial mass="${base_mass}"/>
+        <visual>
+            <geometry>
+                <box size="0.5 0.1 0.1" />
+            </geometry>
+            <material name="red"/>
+        </visual>
+        <collision name = "busted">
+            <geometry>
+                <box size="0.6 0.1 0.1" />
+            </geometry>
+        </collision>
+    </link>
+    <joint name="catch_joint" type="fixed">
+        <parent link="base_link"/>
+        <child link="catch"/>
+        <origin rpy="0 0 0" xyz="0.3 0 -0.35"/>
+    </joint>
     <link name="pols_camera">
         <xacro:default_inertial mass="${eyeball_mass}"/>
